File: KiCAD_Project/PID Demo Board/PID Demo Board.sch (KiCad schematic (older format))
At the start: 44 parts

Commit message: Tweaks and production file creation.
Parts:
- added PCB1: barepcb, misc:barepcb, symbol misc:barepcb
- gave numbers to parts that had none: 41
Other:
- note added: "D Stage"
- note added: "I Stage"
- note added: "Input"
- note added: "Output"
- note added: "P Stage"
- note added: "Power Output"
- moved on the sheet: J1, J3, J4
